File: receiver/receiver.sch (KiCad schematic (older format))
At the start: 22 parts, among them CON1 AVR-ISP-6, IC1 ATTINY85-S, P1 MOTOR, P2 MAIN_BUTTON, P3 MX-05V, P4 LEDs, Q1 S8050, Q2 S8550, Q3 S8550, Q4 S8050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

Commit message: Receiver and transmitter PCB design
Parts:
- removed Q6: S8050, TO_SOT_Packages_THT:TO-92_Inline_Narrow_Oval, symbol Q_NPN_EBC
- removed R7: 220, Resistors_SMD:R_0805_HandSoldering, symbol R
- added Q6: 2N7002, TO_SOT_Packages_SMD:SOT-23_Handsoldering, symbol Q_NMOS_GSD
- Q2, Q3: footprint TO_SOT_Packages_THT:TO-92_Inline_Narrow_Oval -> TO_SOT_Packages_THT:TO-92_Inline_Wide
Connections:
- net GND: now also Q6.2 (S)
- net MCU-LED: now also Q6.1 (G)
- net at R6.2: now also Q6.3 (D)
Changed lines of the file:
@@
 LIBS:contrib
 LIBS:valves
+LIBS:receiver-cache
 EELAYER 25 0
 EELAYER END
@@
 	1    0    0    -1
 $EndComp
-Wire Wire Line
-	10000 1650 10000 1550
-Text Label 9250 1850 2    60   ~ 0
+Text Label 9600 1850 2    60   ~ 0
 MCU-LED
 Wire Wire Line
@@
 F 0 "Q2" H 5450 3600 50  0000 R CNN
 F 1 "S8550" H 5750 3500 50  0000 R CNN
-F 2 "TO_SOT_Packages_THT:TO-92_Inline_Narrow_Oval" H 5350 3650 50  0001 C CNN
+F 2 "TO_SOT_Packages_THT:TO-92_Inline_Wide" H 5350 3650 50  0001 C CNN
 F 3 "" H 5150 3550 50  0000 C CNN
 	1    5150 3550
@@
 F 0 "Q3" H 6700 3600 50  0000 R CNN
 F 1 "S8550" H 7000 3500 50  0000 R CNN
-F 2 "TO_SOT_Packages_THT:TO-92_Inline_Narrow_Oval" H 6600 3650 50  0001 C CNN
+F 2 "TO_SOT_Packages_THT:TO-92_Inline_Wide" H 6600 3650 50  0001 C CNN
 F 3 "" H 6400 3550 50  0000 C CNN
 	1    6400 3550
@@
 	1650 1450 1350 1450
 Connection ~ 1350 1450
-$Comp
-L R R7
-U 1 1 578254A6
-P 9450 1850
-F 0 "R7" V 9530 1850 50  0000 C CNN
-F 1 "220" V 9450 1850 50  0000 C CNN
-F 2 "Resistors_SMD:R_0805_HandSoldering" V 9380 1850 50  0001 C CNN
-F 3 "" H 9450 1850 50  0000 C CNN
-	1    9450 1850
-	0    1    1    0
-$EndComp
-Wire Wire Line
-	9250 1850 9300 1850
-$Comp
-L Q_NPN_EBC Q6
-U 1 1 57825665
-P 9900 1850
-F 0 "Q6" H 10200 1900 50  0000 R CNN
-F 1 "S8050" H 10500 1800 50  0000 R CNN
-F 2 "TO_SOT_Packages_THT:TO-92_Inline_Narrow_Oval" H 10100 1950 50  0001 C CNN
-F 3 "" H 9900 1850 50  0000 C CNN
-	1    9900 1850
-	1    0    0    -1
-$EndComp
 Text Notes 1100 2400 0    60   ~ 0
 programming header
@@
 Text Notes 9450 650  0    60   ~ 0
 lights on the locomotive
+$Comp
+L Q_NMOS_GSD Q6
+U 1 1 578243FE
+P 9900 1850
+F 0 "Q6" H 10200 1900 50  0000 R CNN
+F 1 "2N7002" H 10550 1800 50  0000 R CNN
+F 2 "TO_SOT_Packages_SMD:SOT-23_Handsoldering" H 10100 1950 50  0001 C CNN
+F 3 "" H 9900 1850 50  0000 C CNN
+	1    9900 1850
+	1    0    0    -1
+$EndComp
+Wire Wire Line
+	10000 1550 10000 1650
 $EndSCHEMATC
