File: transmitter/transmitter.sch (KiCad schematic (older format))
At the start: 26 parts, among them CON1 AVR-ISP-6, IC1 ATTINY85-P, P1 9V, P2 MX-FS-03V, Q1 2N7002LT1G, Q2 BSS315, Q3 2N7002LT1G, SW1 FWD, SW2 STOP, SW3 REV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

Commit message: receiver schematics
Parts:
- Q1, Q3: value 2N7002LT1G -> 2N7002
Changed lines of the file:
@@
 P 7100 2100
 F 0 "Q1" H 7400 2150 50  0000 R CNN
-F 1 "2N7002LT1G" H 7750 2050 50  0000 R CNN
+F 1 "2N7002" H 7750 2050 50  0000 R CNN
 F 2 "TO_SOT_Packages_SMD:SOT-23_Handsoldering" H 7300 2200 50  0001 C CNN
 F 3 "" H 7100 2100 50  0000 C CNN
@@
 P 3700 5750
 F 0 "Q3" H 4000 5800 50  0000 R CNN
-F 1 "2N7002LT1G" H 4350 5700 50  0000 R CNN
+F 1 "2N7002" H 4350 5700 50  0000 R CNN
 F 2 "TO_SOT_Packages_SMD:SOT-23_Handsoldering" H 3900 5850 50  0001 C CNN
 F 3 "" H 3700 5750 50  0000 C CNN

Commit message: Receiver and transmitter PCB design
Parts:
- P1: footprint Connect:PINHEAD1-2 -> Pin_Headers:Pin_Header_Straight_1x02
- P2: footprint Connect:PINHEAD1-3 -> Pin_Headers:Pin_Header_Angled_1x03
- U1: footprint Power_Integrations:SO-8 -> TO_SOT_Packages_THT:TO-220_Neutral123_Vertical
Changed lines of the file:
@@
 F 0 "P1" H 1350 1600 50  0000 C CNN
 F 1 "9V" V 1450 1450 50  0000 C CNN
-F 2 "Connect:PINHEAD1-2" H 1350 1450 50  0001 C CNN
+F 2 "Pin_Headers:Pin_Header_Straight_1x02" H 1350 1450 50  0001 C CNN
 F 3 "" H 1350 1450 50  0000 C CNN
 	1    1350 1450
@@
 F 0 "U1" H 3700 1254 50  0000 C CNN
 F 1 "78L05" H 3550 1650 50  0000 C CNN
-F 2 "Power_Integrations:SO-8" H 3550 1450 50  0001 C CNN
+F 2 "TO_SOT_Packages_THT:TO-220_Neutral123_Vertical" H 3550 1450 50  0001 C CNN
 F 3 "" H 3550 1450 50  0000 C CNN
 	1    3550 1450
@@
 F 0 "P2" H 6100 4900 50  0000 C CNN
 F 1 "MX-FS-03V" V 6200 4700 50  0000 C CNN
-F 2 "Connect:PINHEAD1-3" H 6100 4700 50  0001 C CNN
+F 2 "Pin_Headers:Pin_Header_Angled_1x03" H 6100 4700 50  0001 C CNN
 F 3 "" H 6100 4700 50  0000 C CNN
 	1    6100 4700
