File: receiver/sch/receiver.kicad_pcb (KiCad board)
At the start: 2 copper layers, 21 parts, among them CON1 AVR-ISP-6, IC1 ATTINY85-S, P1 MOTOR, P2 MAIN_BUTTON, P3 MX-05V, P4 LEDs, Q1 S8050, Q2 S8550, Q3 S8550, Q4 S8050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

Commit message: organizing files
Other:
- board outline added: 45 x 58 mm
Changed lines of the file:
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@@
   (general
     (links 41)
-    (no_connects 5)
-    (area 143.6318 75.565 187.960001 99.814152)
+    (no_connects 0)
+    (area 69.949999 49.949999 187.960001 108.050001)
     (thickness 1.6)
-    (drawings 0)
+    (drawings 15)
     (tracks 116)
     (zones 0)
@@
     )
   )
+  (gr_circle (center 112 79) (end 112 78) (layer Edge.Cuts) (width 0.1))
+  (gr_line (start 113 83) (end 109 83) (layer Edge.Cuts) (width 0.1))
+  (gr_line (start 115 77) (end 115 81) (layer Edge.Cuts) (width 0.1))
+  (gr_line (start 109 75) (end 113 75) (layer Edge.Cuts) (width 0.1))
+  (gr_arc (start 113 81) (end 115 81) (angle 90) (layer Edge.Cuts) (width 0.1))
+  (gr_arc (start 113 77) (end 113 75) (angle 90) (layer Edge.Cuts) (width 0.1))
+  (gr_line (start 109 64) (end 109 75) (layer Edge.Cuts) (width 0.1))
+  (gr_line (start 109 94) (end 109 83) (layer Edge.Cuts) (width 0.1))
+  (gr_line (start 81 94) (end 109 94) (layer Edge.Cuts) (width 0.1))
+  (gr_line (start 81 64) (end 109 64) (layer Edge.Cuts) (width 0.1))
+  (gr_line (start 81 108) (end 81 94) (layer Edge.Cuts) (width 0.1))
+  (gr_line (start 70 107) (end 81 107) (layer Edge.Cuts) (width 0.1))
+  (gr_line (start 70 50) (end 70 108) (layer Edge.Cuts) (width 0.1))
+  (gr_line (start 81 50) (end 81 64) (layer Edge.Cuts) (width 0.1))
+  (gr_line (start 70 51) (end 81 51) (layer Edge.Cuts) (width 0.1))
   (segment (start 151.765 97.155) (end 151.765 95.554801) (width 0.508) (layer F.Cu) (net 1))
   (via (at 151.765 97.155) (size 2.032) (drill 0.381) (layers F.Cu B.Cu) (net 1))

Commit message: receiver board layout update
Parts:
- C1: moved to F.Cu
- D1: value red -> RX; footprint LEDs:LED-3MM -> LEDs:LED_0805
- P2: value MAIN_BUTTON -> MAIN_BTN
- moved P3 172.4 mm to (24.5, 21.5)
- moved Q5 163.8 mm to (30.2, 21.0)
- moved R5 158.7 mm to (36.5, 21.0), turned to 180 degrees
- moved D1 153.9 mm to (36.7, 21.0), turned to 180 degrees
- moved BT1 152.9 mm to (25.7, 45.2), turned to 270 degrees
- moved P4 150.6 mm to (25.7, 40.1), turned to 270 degrees
- moved R6 149.1 mm to (23.8, 34.4), turned to 270 degrees
- moved IC1 146.0 mm to (34.0, 27.4)
- moved CON1 144.6 mm to (42.9, 25.5)
- moved P2 143.4 mm to (42.9, 21.0)
- moved C1 143.3 mm to (34.0, 26.1)
- moved Q6 140.8 mm to (27.0, 34.4), turned to 0 degrees
- moved R4 138.7 mm to (31.4, 34.2), turned to 180 degrees
- moved R1 133.8 mm to (39.1, 34.2), turned to 180 degrees
- moved Q4 133.1 mm to (32.7, 38.1), turned to 180 degrees
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Connections:
- CON1 pad 1: /MISO -> /MCU-LED
- CON1 pad 4: /MCU-LED -> /MOSI
- IC1 pad 5: /MCU-LED -> /MOSI
- IC1 pad 6: /MISO -> /MCU-LED
- P3 pad 2: /MISO -> /MOSI
- P3 pad 3: /MISO -> /MOSI
- Q5 pad 1: /MISO -> /MOSI
Routing:
- net +5V: track 85.1 -> 2.70 mm, vias 2 -> 1
- net /MOSI: track 0.00 -> 32.6 mm
- net /MISO: track 27.0 -> 0.00 mm
- net Net-(P1-Pad1): track 15.2 -> 29.8 mm
- net GND: track 16.0 -> 27.5 mm, vias 0 -> 1
- net /MOT_A: track 2.93 -> 10.6 mm
- net /MOT_B: track 2.93 -> 10.4 mm
- net /MCU-LED: track 31.5 -> 26.2 mm, vias 2 -> 0
- net Net-(P4-Pad2): track 3.09 -> 8.17 mm
- net /RST: track 17.3 -> 13.2 mm, vias 0 -> 1
- net Net-(Q6-Pad3): track 7.30 -> 3.24 mm
- net Net-(P1-Pad2): track 25.9 -> 24.1 mm
- net /MAIN_BUTTON: track 12.7 -> 13.3 mm
- net Net-(D1-Pad1): track 3.65 -> 4.26 mm, vias 0 -> 1
- added copper zone on F.Cu, net +5V
Other:
- board size 45 x 58 mm -> 35 x 30 mm
- net class Default: clearance 0.2032 -> 0.254; via_dia 2.032 -> 1.27
- rule trace_clearance: 0.2032 -> 0.254
- rule trace_min: 0.2 -> 0.254
- rule via_min_size: 0.4 -> 1.016
- board text added: "LEGO Duplo locomotive controller Simon Fojtu 2016 rev. 1"

Commit message: receiver pcb rev.1
Parts:
- added P5: mounting hole, Mounting_Holes:MountingHole_3.5mm_Pad, F.Cu at (52.0, 34.0)
- D1: value RX -> red
- P2: value MAIN_BTN -> MAIN_BUTTON
Other:
- outline, holes or cut-outs redrawn
Changed lines of the file:
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@@
   (general
     (links 41)
-    (no_connects 1)
-    (area 79.949999 63.949999 115.050001 94.050001)
+    (no_connects 0)
+    (area 19.949999 18.949999 55.050001 49.050001)
     (thickness 1.6)
-    (drawings 12)
+    (drawings 11)
     (tracks 95)
     (zones 0)
-    (modules 21)
+    (modules 22)
     (nets 19)
   )
@@
       (effects (font (size 1 1) (thickness 0.15)))
     )
-    (fp_text value MAIN_BTN (at 1.13 1.96) (layer F.Fab)
+    (fp_text value MAIN_BUTTON (at 1.13 1.96) (layer F.Fab)
       (effects (font (size 1 1) (thickness 0.15)))
     )
@@
       (effects (font (size 1 1) (thickness 0.15)))
     )
-    (fp_text value RX (at 3.74098 1.04 180) (layer F.Fab)
+    (fp_text value red (at 3.74098 1.04 180) (layer F.Fab)
       (effects (font (size 1 1) (thickness 0.15)))
     )
@@
     )
   )
+  (module Mounting_Holes:MountingHole_3.5mm_Pad (layer F.Cu)
+    (at 52 34)
+    (descr "Mounting Hole 3.5mm")
+    (tags "mounting hole 3.5mm")
+    (fp_text reference P5 (at 0 -4.5) (layer F.SilkS)
+      (effects (font (size 1 1) (thickness 0.15)))
+    )
+    (fp_text value "mounting hole" (at 0 4.5) (layer F.Fab)
+      (effects (font (size 1 1) (thickness 0.15)))
+    )
+    (fp_circle (center 0 0) (end 3.5 0) (layer Cmts.User) (width 0.15))
+    (fp_circle (center 0 0) (end 3.75 0) (layer F.CrtYd) (width 0.05))
+    (pad 1 thru_hole circle (at 0 0) (size 7 7) (drill 3.5) (layers *.Cu *.Mask F.SilkS))
+  )
   (gr_text "LEGO Duplo locomotive controller\nSimon Fojtu 2016\nrev. 1" (at 21.915 35.01) (layer F.SilkS)
     (effects (font (size 0.762 0.762) (thickness 0.127)) (justify left))
   )
-  (gr_circle (center 52 34) (end 52 32) (layer Edge.Cuts) (width 0.1))
   (gr_line (start 20 49) (end 20 19) (layer Edge.Cuts) (width 0.1))
   (gr_line (start 53 38) (end 49 38) (layer Edge.Cuts) (width 0.1))
