File: receiver/sch/receiver.sch (KiCad schematic (older format))
At the start: 21 parts, among them CON1 AVR-ISP-6, IC1 ATTINY85-S, P1 MOTOR, P2 MAIN_BUTTON, P3 MX-05V, P4 LEDs, Q1 S8050, Q2 S8550, Q3 S8550, Q4 S8050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

Commit message: receiver board layout update
Parts:
- D1: footprint LEDs:LED-3MM -> LEDs:LED_0805
- P3: footprint Pin_Headers:Pin_Header_Straight_1x04 -> Pin_Headers:Pin_Header_Angled_1x04
Connections:
- net MCU-LED: now also CON1.1, IC1.6 (PB1(MISO/DO/AIN1/OC0B/OC1A/PCINT1)); no longer CON1.4, IC1.5 (PB0(MOSI/DI/SDA/AIN0/OC0A/OC1A/AREF/PCINT0))
- net MISO renamed MOSI
- net MOSI: now also CON1.4, IC1.5 (PB0(MOSI/DI/SDA/AIN0/OC0A/OC1A/AREF/PCINT0)); no longer CON1.1, IC1.6 (PB1(MISO/DO/AIN1/OC0B/OC1A/PCINT1))
Changed lines of the file:
@@
 Wire Wire Line
 	9600 1850 9700 1850
-Text Label 2550 1150 0    60   ~ 0
+Text Label 2550 1250 0    60   ~ 0
 MCU-LED
 Text Label 3550 1250 0    60   ~ 0
@@
 F 0 "P3" H 1900 4250 50  0000 C CNN
 F 1 "MX-05V" V 2000 4000 50  0000 C CNN
-F 2 "Pin_Headers:Pin_Header_Straight_1x04" H 1900 4000 50  0001 C CNN
+F 2 "Pin_Headers:Pin_Header_Angled_1x04" H 1900 4000 50  0001 C CNN
 F 3 "" H 1900 4000 50  0000 C CNN
 	1    1900 4000
@@
 RX-DATA
 Connection ~ 1600 3950
-Text Label 2550 1250 0    60   ~ 0
+Text Label 2550 1150 0    60   ~ 0
 RX-DATA
 $Comp
@@
 F 0 "D1" H 10000 3550 50  0000 C CNN
 F 1 "red" H 10000 3350 50  0000 C CNN
-F 2 "LEDs:LED-3MM" H 10000 3450 50  0001 C CNN
+F 2 "LEDs:LED_0805" H 10000 3450 50  0001 C CNN
 F 3 "" H 10000 3450 50  0000 C CNN
 	1    10000 3450

Commit message: receiver pcb rev.1
Parts:
- added P?: mounting hole, symbol CONN_01X01
- P3: footprint Pin_Headers:Pin_Header_Angled_1x04 -> Pin_Headers:Pin_Header_Straight_1x04
Connections:
- no-connect marks 0 -> 1
Changed lines of the file:
@@
 F 0 "P3" H 1900 4250 50  0000 C CNN
 F 1 "MX-05V" V 2000 4000 50  0000 C CNN
-F 2 "Pin_Headers:Pin_Header_Angled_1x04" H 1900 4000 50  0001 C CNN
+F 2 "Pin_Headers:Pin_Header_Straight_1x04" H 1900 4000 50  0001 C CNN
 F 3 "" H 1900 4000 50  0000 C CNN
 	1    1900 4000
@@
 Wire Wire Line
 	10000 1550 10000 1650
+$Comp
+L CONN_01X01 P?
+U 1 1 578DF3F0
+P 7500 5800
+F 0 "P?" H 7500 5900 50  0000 C CNN
+F 1 "mounting hole" V 7600 5800 50  0000 C CNN
+F 2 "" H 7500 5800 50  0000 C CNN
+F 3 "" H 7500 5800 50  0000 C CNN
+	1    7500 5800
+	0    1    1    0
+$EndComp
+NoConn ~ 7500 5600
 $EndSCHEMATC
